File: schemes/electronics/Circuito/Circuito.sch (EAGLE design)
At the start: 20 parts, among them IC1 ARD-NANO30NP, U1 ESP32-DEV-KIT-V1

Commit message: Add files via upload
Circuito 2.1
Parts:
- removed L298N: (no value), con-amp-quick:L298N
- removed MOTOR: (no value), ngspice-simulation:VOLTAGE
- added D3, D4: U57X32, led:U57X32
- added IC3: ARD-NANO30NP, ARD-NANO30NP:ARD-NANO30NP
- added IC4: (no value), v-reg:78XXS
- added MOTOR1: (no value), ngspice-simulation:VOLTAGE
- added SERVO2: (no value), con-amp-quick:CON_SERVO
- added SL2, SL3, SL4: (no value), con-amp-quick:M03
- added TB1, TB2: TB6612FNG, TB6612FNG:TB6612FNG
- added ULTRA_CENTRO1: (no value), con-amp-quick:M04
Connections:
- removed net ECHO_D4: IC1.D4, ULTRA_CENTRO.2
- removed net ECHO_D6: IC1.D6, ULTRA_DERECHO.2
- removed net N$6: L298N.12, L298N.2, MOTOR.+
- removed net N$7: L298N.1, L298N.13, MOTOR.-
- removed net TIGGER_D5: IC1.D5, ULTRA_CENTRO.3
- removed net TIGGER_D7: IC1.D7, ULTRA_DERECHO.3
- new net ECHO_F6: ULTRA_CENTRO.2
- new net ECHO_I4: ULTRA_IZQUIERDO.2
- new net ECHO_T15: ULTRA_CENTRO1.2
- new net N$14: IC1.A1
- new net N$15: IC3.D3
- new net N$16: U1.D33
- new net N$17: TB1.VM, TB2.VM
- new net N$18: TB1.VCC, TB2.VCC
- new net N$2: IC1.D3
- new net N$21: MOTOR1.-, TB1.A2, TB1.B2, TB2.A2, TB2.B2
- new net N$23: MOTOR1.+, TB1.A1, TB1.B1, TB2.A1, TB2.B1
- new net N$4: IC1.D8
- new net N$8: IC1.D13
- new net OUT_C: SL3.SEÑAL
- new net OUT_D: SL2.SEÑAL
- new net OUT_I: SL4.SEÑAL
- new net PMOTOR: IC1.D5, TB1.PWMA, TB1.PWMB, TB2.PWMA, TB2.PWMB
- new net SEÑAL_SERVO_CAM: SERVO2.SEÑAL
- new net TIGGER_F7: ULTRA_CENTRO.3
- new net TIGGER_I11: ULTRA_IZQUIERDO.3
- new net TRIGGER_T13: ULTRA_CENTRO1.3
- new net V5V: SL2.5V, SL3.5V
- net 5VBAT: now also D4.A, IC4.OUT
- net DIR1: now also IC1.A2, TB1.AIN1, TB1.BIN1, TB2.AIN1, TB2.BIN1; no longer IC1.A1, L298N.7, L298N.9
- net DIR2: now also IC1.A3, TB1.AIN2, TB1.BIN2, TB2.AIN2, TB2.BIN2; no longer IC1.A2, L298N.10, L298N.8
- net ECHO_D8: now also ULTRA_DERECHO.2; no longer IC1.D8, ULTRA_IZQUIERDO.2
- net ENA: now also IC1.A0, TB1.STBY, TB2.STBY; no longer IC1.D11, L298N.11, L298N.6
- net GND: now also IC4.GND, SERVO2.GND, SL2.GND, SL3.GND, SL4.GND, TB1.GND1, TB1.GND2, TB1.GND3, TB2.GND1, TB2.GND2, TB2.GND3, ULTRA_CENTRO1.4; no longer L298N.4
- net TIGGER_D3: now also ULTRA_DERECHO.3; no longer IC1.D3, ULTRA_IZQUIERDO.3
- net VBAT: now also D3.A, IC4.IN; no longer L298N.3
- net VCC_5V_SERVO: now also SERVO2.5V, ULTRA_CENTRO1.1
Other:
- note added: "Circuito del Robot del Equipo de Gammaversion"
- note added: "Drivers del Motor y Motor"
- note added: "Fuente de Alimentación de los Servos"
- note added: "Nano 2"
- note added: "Sensor Laser Central"
- note added: "Sensor Laser Derecho"
- note added: "Sensor Laser Izquierdo"
- note added: "Servo Camara"
- note added: "Ultrasonido Frontal"
- note added: "Ultrasonido Tracero"
- note removed: "Driver del Motor y Motor"
- note removed: "Ultrasonido Central"
- moved on the sheet: ULTRA_DERECHO, ULTRA_IZQUIERDO
